Commit message: Added rviz visuallization

File: yeti_snowplow/models/yeti/model.urdf (robot description, URDF)
Before this commit: robot yeti, 5 links, 4 joints
Links:
- removed link chassis
- added link base_link; visual box size=.93 .495 .625
Joints:
- joint left_back_wheel_hinge: parent chassis -> base_link
- joint left_front_wheel_hinge: parent chassis -> base_link
- joint right_back_wheel_hinge: parent chassis -> base_link
- joint right_front_wheel_hinge: parent chassis -> base_link
